Commit message: Add files via upload
Fixed the origin problem of the axis

File: robotont_description/urdf/robotont_description.urdf (robot description, URDF)
Before this commit: robot robotont_description, 46 links, 45 joints
Links:
- link Omniwheel1: mass 0.022436 -> 0.0224355329965772; geometry collision mesh filename=package://robotont_description/meshes/Omniwheel1.STL; visual mesh filename=package://robotont_description/meshes/Omniwheel1.STL
- link Omniwheel2: mass 0.022435522293739 -> 0.0224355229928124; geometry collision mesh filename=package://robotont_description/meshes/Omniwheel2.STL; visual mesh filename=package://robotont_description/meshes/Omniwheel2.STL
- link Omniwheel3: mass 0.0224355450669598 -> 0.0224355457660329; geometry collision mesh filename=package://robotont_description/meshes/Omniwheel3.STL; visual mesh filename=package://robotont_description/meshes/Omniwheel3.STL
- link Roller11: geometry collision mesh filename=package://robotont_description/meshes/Roller11.STL; visual mesh filename=package://robotont_description/meshes/Roller11.STL
- link Roller110: geometry collision mesh filename=package://robotont_description/meshes/Roller110.STL; visual mesh filename=package://robotont_description/meshes/Roller110.STL
- link Roller111: geometry collision mesh filename=package://robotont_description/meshes/Roller111.STL; visual mesh filename=package://robotont_description/meshes/Roller111.STL
- link Roller112: geometry collision mesh filename=package://robotont_description/meshes/Roller112.STL; visual mesh filename=package://robotont_description/meshes/Roller112.STL
- link Roller113: geometry collision mesh filename=package://robotont_description/meshes/Roller113.STL; visual mesh filename=package://robotont_description/meshes/Roller113.STL
- link Roller114: geometry collision mesh filename=package://robotont_description/meshes/Roller114.STL; visual mesh filename=package://robotont_description/meshes/Roller114.STL
- link Roller12: geometry collision mesh filename=package://robotont_description/meshes/Roller12.STL; visual mesh filename=package://robotont_description/meshes/Roller12.STL
- link Roller13: geometry collision mesh filename=package://robotont_description/meshes/Roller13.STL; visual mesh filename=package://robotont_description/meshes/Roller13.STL
- link Roller14: geometry collision mesh filename=package://robotont_description/meshes/Roller14.STL; visual mesh filename=package://robotont_description/meshes/Roller14.STL
- link Roller15: geometry collision mesh filename=package://robotont_description/meshes/Roller15.STL; visual mesh filename=package://robotont_description/meshes/Roller15.STL
- link Roller16: geometry collision mesh filename=package://robotont_description/meshes/Roller16.STL; visual mesh filename=package://robotont_description/meshes/Roller16.STL
- link Roller17: geometry collision mesh filename=package://robotont_description/meshes/Roller17.STL; visual mesh filename=package://robotont_description/meshes/Roller17.STL
- link Roller18: geometry collision mesh filename=package://robotont_description/meshes/Roller18.STL; visual mesh filename=package://robotont_description/meshes/Roller18.STL
- link Roller19: geometry collision mesh filename=package://robotont_description/meshes/Roller19.STL; visual mesh filename=package://robotont_description/meshes/Roller19.STL
- link Roller21: geometry collision mesh filename=package://robotont_description/meshes/Roller21.STL; visual mesh filename=package://robotont_description/meshes/Roller21.STL
- link Roller210: geometry collision mesh filename=package://robotont_description/meshes/Roller210.STL; visual mesh filename=package://robotont_description/meshes/Roller210.STL
- link Roller211: geometry collision mesh filename=package://robotont_description/meshes/Roller211.STL; visual mesh filename=package://robotont_description/meshes/Roller211.STL
- link Roller212: geometry collision mesh filename=package://robotont_description/meshes/Roller212.STL; visual mesh filename=package://robotont_description/meshes/Roller212.STL
- link Roller213: mass 0.00222805342991147 -> 0.00222805342991146; geometry collision mesh filename=package://robotont_description/meshes/Roller213.STL; visual mesh filename=package://robotont_description/meshes/Roller213.STL
- link Roller214: geometry collision mesh filename=package://robotont_description/meshes/Roller214.STL; visual mesh filename=package://robotont_description/meshes/Roller214.STL
- link Roller22: geometry collision mesh filename=package://robotont_description/meshes/Roller22.STL; visual mesh filename=package://robotont_description/meshes/Roller22.STL
- link Roller23: geometry collision mesh filename=package://robotont_description/meshes/Roller23.STL; visual mesh filename=package://robotont_description/meshes/Roller23.STL
- link Roller24: geometry collision mesh filename=package://robotont_description/meshes/Roller24.STL; visual mesh filename=package://robotont_description/meshes/Roller24.STL
- link Roller25: geometry collision mesh filename=package://robotont_description/meshes/Roller25.STL; visual mesh filename=package://robotont_description/meshes/Roller25.STL
- link Roller26: mass 0.00222805035043754 -> 0.0022281; geometry collision mesh filename=package://robotont_description/meshes/Roller26.STL; visual mesh filename=package://robotont_description/meshes/Roller26.STL
- link Roller27: geometry collision mesh filename=package://robotont_description/meshes/Roller27.STL; visual mesh filename=package://robotont_description/meshes/Roller27.STL
- link Roller28: geometry collision mesh filename=package://robotont_description/meshes/Roller28.STL; visual mesh filename=package://robotont_description/meshes/Roller28.STL
- link Roller29: geometry collision mesh filename=package://robotont_description/meshes/Roller29.STL; visual mesh filename=package://robotont_description/meshes/Roller29.STL
- link Roller31: geometry collision mesh filename=package://robotont_description/meshes/Roller31.STL; visual mesh filename=package://robotont_description/meshes/Roller31.STL
- link Roller310: geometry collision mesh filename=package://robotont_description/meshes/Roller310.STL; visual mesh filename=package://robotont_description/meshes/Roller310.STL
- link Roller311: geometry collision mesh filename=package://robotont_description/meshes/Roller311.STL; visual mesh filename=package://robotont_description/meshes/Roller311.STL
- link Roller312: geometry collision mesh filename=package://robotont_description/meshes/Roller312.STL; visual mesh filename=package://robotont_description/meshes/Roller312.STL
- link Roller313: geometry collision mesh filename=package://robotont_description/meshes/Roller313.STL; visual mesh filename=package://robotont_description/meshes/Roller313.STL
- link Roller314: geometry collision mesh filename=package://robotont_description/meshes/Roller314.STL; visual mesh filename=package://robotont_description/meshes/Roller314.STL
- link Roller32: geometry collision mesh filename=package://robotont_description/meshes/Roller32.STL; visual mesh filename=package://robotont_description/meshes/Roller32.STL
- link Roller33: geometry collision mesh filename=package://robotont_description/meshes/Roller33.STL; visual mesh filename=package://robotont_description/meshes/Roller33.STL
- link Roller34: geometry collision mesh filename=package://robotont_description/meshes/Roller34.STL; visual mesh filename=package://robotont_description/meshes/Roller34.STL
- link Roller35: geometry collision mesh filename=package://robotont_description/meshes/Roller35.STL; visual mesh filename=package://robotont_description/meshes/Roller35.STL
- link Roller36: geometry collision mesh filename=package://robotont_description/meshes/Roller36.STL; visual mesh filename=package://robotont_description/meshes/Roller36.STL
- link Roller37: geometry collision mesh filename=package://robotont_description/meshes/Roller37.STL; visual mesh filename=package://robotont_description/meshes/Roller37.STL
- link Roller38: geometry collision mesh filename=package://robotont_description/meshes/Roller38.STL; visual mesh filename=package://robotont_description/meshes/Roller38.STL
- link Roller39: geometry collision mesh filename=package://robotont_description/meshes/Roller39.STL; visual mesh filename=package://robotont_description/meshes/Roller39.STL
- link base_link: mass 0.8967 -> 0.896698981932657; geometry collision mesh filename=package://robotont_description/meshes/base_link.STL; visual mesh filename=package://robotont_description/meshes/base_link.STL
Joints:
- joint Roller11: origin xyz=0 0.0017898 -0.0017588 rpy=0.36277 4.996E-16 -2.2204E-16 -> xyz=-0.00905600884677152 0.0275059261982972 0.00800224940532278 rpy=0.362770953244145 -2.22044604925031E-16 1.0547118733939E-15
- joint Roller110: axis 1 0 0 -> 0.999999999218083 0 3.95453473158447E-05; origin xyz=0.0431432440899406 0.00984716392754997 -0.0298081468021298 rpy=0.915756259459611 -2.22044604925031E-16 1.7951958020513 -> xyz=0.0288219044427726 -0.0027104893795199 -0.00799497322847986 rpy=0.915756259837358 2.40906703969355E-05 1.79522716244185
- joint Roller111: axis 1 0 0 -> 0.999999999804521 0 1.97726715280566E-05; origin xyz=0.0345981954807621 -0.0275911401992598 -0.0298081468021298 rpy=0.915756259459612 -3.33066907387547E-16 0.897597901025643 -> xyz=0.0158510175604117 -0.0242238347642219 -0.00799497322847989 rpy=0.915756259554049 1.20453338984942E-05 0.897613581219221
- joint Roller112: origin xyz=0 -0.0442527529993359 -0.0298081468021298 rpy=0.915756259459611 1.11022302462516E-16 9.43689570931383E-16 -> xyz=-0.00905600884677145 -0.0274961384952869 -0.00799497322847989 rpy=0.915756259459612 -2.77555756156289E-16 1.22124532708767E-15
- joint Roller113: origin xyz=-0.0345981954807624 -0.0275911401992594 -0.0298081468021298 rpy=0.915756259459614 -1.38777878078145E-17 -0.897597901025655 -> xyz=-0.0271436758834209 -0.0100632891203918 -0.00799497322847989 rpy=0.915756259459612 1.94289029309402E-16 -0.897597901025656
- joint Roller114: axis -1 0 0 -> -0.999999995113017 0 -9.88633677644346E-05; origin xyz=-0.0431432440899404 0.00984716392755047 -0.0298081468021298 rpy=0.915756259459612 1.38777878078145E-15 -1.79519580205131 -> xyz=-0.024791601349772 0.0149474222158465 -0.00799497322847989 rpy=0.915756261820527 6.02266757044277E-05 -1.79511740107518
- joint Roller12: axis -1 0 0 -> -0.99999999859084 0 -5.30878583583499E-05; origin xyz=0 0.00178977984606152 -0.00175882060681612 rpy=0.362770953244145 1.33226762955019E-15 -0.897597901025656 -> xyz=0.0158586698947665 0.0242299372972322 0.00800224940532278 rpy=0.362770953711663 4.96327464162194E-05 -0.897579061938864
- joint Roller13: axis -1 0 0 -> -0.999999999021416 0 -4.42398835954205E-05; origin xyz=0.0013993062303377 0.00111590948159165 -0.00175882060681612 rpy=0.362770953244145 8.88178419700125E-16 -1.79519580205131 -> xyz=0.0288314467476335 0.00270831141070441 0.00800224940532276 rpy=0.362770953568811 4.136062353274E-05 -1.79518010281175
- joint Roller14: axis 1 0 0 -> 0.999999999373706 0 3.53919053181495E-05; origin xyz=0 0 0 rpy=0.362770953244144 -1.66533453693773E-16 -2.69279370307697 -> xyz=0.0200935561451987 -0.0208527282075686 0.00800224940532276 rpy=0.36277095345193 3.30884973664274E-05 -2.69278114368587
- joint Roller15: axis 1 0 0 -> 0.99999999964771 0 2.65439304654308E-05; origin xyz=0.000776556371806431 -0.00161253592170063 -0.00175882060681613 rpy=0.362770953244145 2.35922392732846E-16 2.69279370307696 -> xyz=-0.00377519206841899 -0.0287112381674063 0.00800224940532274 rpy=0.362770953361024 2.48163744035266E-05 2.6928031226208
- joint Roller16: axis 1 0 0 -> 0.999999999843426 0 1.76959534931714E-05; origin xyz=-0.000776556371806417 -0.0016125359217006 -0.00175882060681613 rpy=0.362770953244145 -5.82867087928207E-16 1.7951958020513 -> xyz=-0.0248011436546332 -0.0149496001846614 0.00800224940532276 rpy=0.362770953296091 1.65442494603261E-05 1.79520208174714
- joint Roller17: axis 1 0 0 -> -0.222517872822441 0.911476772960516 -0.345970936103106; origin xyz=0 0.00178977984606152 -0.00175882060681612 rpy=0.362770953244145 -1.11022302462516E-15 0.897597901025643 -> xyz=-0.0271513282177754 0.0100693916534027 0.00800224940532278 rpy=0.362770953257132 8.27212416175113E-06 0.897601040873349
- joint Roller18: axis 1 0 0 -> 0.999999996872331 0 7.90906943926584E-05; origin xyz=-0.019201 0.03987 -0.029808 rpy=0.91576 -4.4409E-16 -2.6928 -> xyz=-0.00377094534323913 0.0287024197517056 -0.00799497322847986 rpy=0.915756260970597 4.81813406636344E-05 -2.69273098229598
- joint Roller19: axis 1 0 0 -> 0.999999998240686 0 5.93180200797877E-05; origin xyz=0.0192005499375979 0.0398703527713769 -0.0298081468021298 rpy=0.915756259459612 -4.71844785465692E-16 2.69279370307696 -> xyz=0.0200893094200195 0.0208439097918678 -0.00799497322847988 rpy=0.915756260309541 3.61360050554162E-05 2.69284074366209
- joint Roller21: origin xyz=0 0 0 rpy=0.362770953244147 2.77555756156289E-16 -7.7715611723761E-16 -> xyz=-0.00905600884677153 0.0275059261982972 0.00800224940532274 rpy=0.362770953244145 0 1.11022302462516E-15
- joint Roller210: origin xyz=0.0431432440899406 0.00984716392754997 -0.0298081468021298 rpy=0.915756259459611 1.38777878078145E-16 1.7951958020513 -> xyz=0.0288219044427726 -0.00271048937951987 -0.00799497322847992 rpy=0.915756259459612 2.77555756156289E-17 1.7951958020513
- joint Roller211: origin xyz=0.0345981954807621 -0.0275911401992598 -0.0298081468021298 rpy=0.915756259459612 -6.86950496486816E-16 0.897597901025644 -> xyz=0.0158510175604116 -0.0242238347642219 -0.00799497322847992 rpy=0.915756259459612 -3.46944695195361E-18 0.897597901025644
- joint Roller212: origin xyz=0 -0.0442527529993359 -0.0298081468021298 rpy=0.915756259459612 5.55111512312578E-17 9.43689570931383E-16 -> xyz=-0.00905600884677145 -0.0274961384952869 -0.00799497322847992 rpy=0.915756259459612 2.77555756156289E-17 1.11022302462516E-15
- joint Roller213: origin xyz=-0.0345981954807624 -0.0275911401992594 -0.0298081468021298 rpy=0.915756259459612 -1.1518563880486E-15 -0.897597901025656 -> xyz=-0.0271436758834209 -0.0100632891203917 -0.00799497322847992 rpy=0.915756259459612 8.32667268468867E-17 -0.897597901025656
- joint Roller214: axis -1 0 0 -> -0.999999995113017 0 -9.88633677652673E-05; origin xyz=-0.0431432440899405 0.00984716392755047 -0.0298081468021298 rpy=0.915756259459611 1.94289029309402E-16 -1.79519580205131 -> xyz=-0.0247916013497721 0.0149474222158466 -0.00799497322847992 rpy=0.915756261820527 6.02266757040028E-05 -1.79511740107518
- joint Roller22: axis -1 0 0 -> -0.99999999859084 0 -5.30878583579128E-05; origin xyz=0 0 0 rpy=0.362770953244146 4.09394740330527E-16 -0.897597901025656 -> xyz=0.0158586698947665 0.0242299372972323 0.00800224940532274 rpy=0.362770953711663 4.96327464161286E-05 -0.897579061938864
- joint Roller23: axis -1 0 0 -> -0.999999999021416 0 -4.42398835952817E-05; origin xyz=0.00139930623033767 0.00111590948159168 -0.00175882060681615 rpy=0.362770953244146 2.77555756156289E-17 -1.79519580205131 -> xyz=0.0288314467476335 0.00270831141070441 0.00800224940532274 rpy=0.36277095356881 4.13606235323142E-05 -1.79518010281175
- joint Roller24: axis -1 0 0 -> -0.999999999373707 0 -3.53919053184271E-05; origin xyz=0 0 0 rpy=0.362770953244146 -3.88578058618805E-16 -2.69279370307697 -> xyz=0.0200935561451987 -0.0208527282075686 0.00800224940532274 rpy=0.362770953451931 3.30884973659497E-05 -2.69278114368587
- joint Roller25: axis 1 0 0 -> 0.99999999964771 0 2.65439304655279E-05; origin xyz=0.000776556371806417 -0.00161253592170063 -0.00175882060681615 rpy=0.362770953244146 -2.22044604925031E-16 2.69279370307696 -> xyz=-0.00377519206841903 -0.0287112381674063 0.00800224940532274 rpy=0.362770953361025 2.48163744033955E-05 2.6928031226208
- joint Roller26: origin xyz=0 0.00178977984606152 -0.00175882060681615 rpy=0.362770953244146 -4.99600361081321E-16 1.7951958020513 -> xyz=-0.0248011436546332 -0.0149496001846614 0.00800224940532274 rpy=0.362770953244145 2.77555756156289E-17 1.7951958020513
- joint Roller27: axis 1 0 0 -> 0.999999999960857 0 0; origin xyz=0 0 0 rpy=0.362770953244147 1.31838984174237E-16 0.897597901025644 -> xyz=-0.0271513282177754 0.0100693916534027 0.00800224940532274 rpy=0.362770953257132 8.27212416226734E-06 0.897601040873349
- joint Roller28: axis -1 0 0 -> -0.999999996872331 0 -7.90906943937686E-05; origin xyz=-0.019201 0.03987 -0.029808 rpy=0.91576 -9.992E-16 -2.6928 -> xyz=-0.00377094534323914 0.0287024197517057 -0.00799497322847992 rpy=0.915756260970598 4.81813406631331E-05 -2.69273098229598
- joint Roller29: axis 1 0 0 -> 0.999999998240686 0 5.93180200794685E-05; origin xyz=0.0192005499375979 0.039870352771377 -0.0298081468021298 rpy=0.915756259459612 -8.60422844084496E-16 2.69279370307696 -> xyz=0.0200893094200194 0.0208439097918678 -0.00799497322847992 rpy=0.915756260309541 3.61360050552819E-05 2.69284074366209
- joint Roller31: origin xyz=0 0 0 rpy=0.362770953244145 2.22044604925031E-16 7.21644966006352E-16 -> xyz=-0.00905600884677155 0.0275059261982972 0.00800224940532271 rpy=0.362770953244144 -1.11022302462516E-16 1.33226762955019E-15
- joint Roller310: axis 1 0 0 -> 0.999999999218083 0 3.95453473166496E-05; origin xyz=0.0431432440899405 0.00984716392754993 -0.0298081468021298 rpy=0.91575625945961 8.32667268468867E-17 1.7951958020513 -> xyz=0.0288219044427725 -0.0027104893795199 -0.00799497322847992 rpy=0.915756259837358 2.40906703979625E-05 1.79522716244185
- joint Roller311: axis -1 0 0 -> -0.999999999804521 0 -1.97726715267521E-05; origin xyz=0.034598195480762 -0.0275911401992598 -0.0298081468021298 rpy=0.915756259459612 1.33226762955019E-15 0.897597901025644 -> xyz=0.0158510175604116 -0.0242238347642219 -0.00799497322847988 rpy=0.915756259554048 1.20453338996044E-05 0.897613581219221
- joint Roller312: origin xyz=0 -0.044252752999336 -0.0298081468021297 rpy=0.915756259459611 5.55111512312578E-16 1.22124532708767E-15 -> xyz=-0.00905600884677144 -0.0274961384952869 -0.00799497322847989 rpy=0.915756259459611 -1.11022302462516E-16 1.27675647831893E-15
- joint Roller313: origin xyz=-0.0215003657678708 -0.0171459695511152 -0.00799999999999999 rpy=-0.422962332618568 -4.16333634234434E-17 -0.897597901025655 -> xyz=-0.027143675883421 -0.0100632891203918 -0.00799497322847988 rpy=0.915756259459612 -5.96744875736022E-16 -0.897597901025656
- joint Roller314: axis 1 0 0 -> 0.999999995113017 0 9.88633677658605E-05; origin xyz=-0.0431432440899405 0.0098471639275504 -0.0298081468021298 rpy=0.915756259459611 2.77555756156289E-16 -1.79519580205131 -> xyz=-0.0247916013497721 0.0149474222158465 -0.00799497322847988 rpy=0.915756261820527 6.02266757033729E-05 -1.79511740107518
- joint Roller32: axis -1 0 0 -> -0.99999999859084 0 -5.30878583584436E-05; origin xyz=0 0 0 rpy=0.362770953244145 -1.33226762955019E-15 -0.897597901025657 -> xyz=0.0167019792096861 0.0253504825559626 0.010944921054306 rpy=0.362770953711663 4.96327464154839E-05 -0.897579061938864
- joint Roller33: axis 1 0 0 -> 0.999999999021417 0 4.42398835973912E-05; origin xyz=0.00139930623033768 0.00111590948159165 -0.00175882060681615 rpy=0.362770953244146 4.44089209850063E-16 -1.79519580205131 -> xyz=0.0288314467476335 0.00270831141070442 0.00800224940532276 rpy=0.36277095356881 4.13606235316853E-05 -1.79518010281175
- joint Roller34: axis 1 0 0 -> 0.999999999373707 0 3.53919053182605E-05; origin xyz=0.0017449 -0.00039826 -0.0017588 rpy=0.36277 4.996E-16 -2.6928 -> xyz=0.0200935561451987 -0.0208527282075686 0.00800224940532279 rpy=0.362770953451931 3.30884973658167E-05 -2.69278114368587
- joint Roller35: axis 1 0 0 -> 0.99999999964771 0 2.65439304664439E-05; origin xyz=0.000776556371806403 -0.00161253592170063 -0.00175882060681615 rpy=0.362770953244146 7.07767178198537E-16 2.69279370307696 -> xyz=-0.00377519206841903 -0.0287112381674062 0.00800224940532276 rpy=0.362770953361025 2.48163744038319E-05 2.6928031226208
- joint Roller36: axis 1 0 0 -> 0.999999999843427 0 1.76959534889387E-05; origin xyz=0 0 0 rpy=0.362770953244147 -6.66133814775094E-16 1.7951958020513 -> xyz=-0.0248011436546332 -0.0149496001846614 0.00800224940532274 rpy=0.362770953296091 1.65442494612698E-05 1.79520208174714
- joint Roller37: axis -1 0 0 -> -0.999999999960857 0 0; origin xyz=0 0 0 rpy=0.362770953244145 9.99200722162641E-16 0.897597901025646 -> xyz=-0.0271513282177754 0.0100693916534027 0.00800224940532274 rpy=0.362770953257131 8.27212416263931E-06 0.897601040873349
- joint Roller38: axis 1 0 0 -> 0.999999996872331 0 7.90906943933245E-05; origin xyz=-0.0192005499375975 0.0398703527713771 -0.0298081468021298 rpy=0.915756259459614 -3.33066907387547E-16 -2.69279370307697 -> xyz=-0.00377094534323918 0.0287024197517056 -0.00799497322847989 rpy=0.915756260970598 4.81813406629683E-05 -2.69273098229598
- joint Roller39: axis 1 0 0 -> 0.999999998240686 0 5.9318020079635E-05; origin xyz=0.0192005499375978 0.0398703527713769 -0.0298081468021298 rpy=0.915756259459612 -4.16333634234434E-16 2.69279370307696 -> xyz=0.0200893094200194 0.0208439097918677 -0.00799497322847993 rpy=0.915756260309542 3.61360050556799E-05 2.69284074366209

Commit message: updated robot_description and added few failsafe checks

File: robotont_description/urdf/robotont_description.urdf (robot description, URDF)
Before this commit: robot test, 46 links, 45 joints
Links:
- added link base_base_link
Joints:
- added joint base_joint: type fixed, parent base_base_link, child base_link, origin xyz=0.254330578207179 0.135454608912068 -0.19184296731081 rpy=0 0 -1.579

Commit message: added camera link to the urdf

File: robotont_description/urdf/robotont_description.urdf (robot description, URDF)
Before this commit: robot test, 47 links, 46 joints
Links:
- added link camera_link
Joints:
- added joint camera_joint: type fixed, parent base_base_link, child camera_link, origin xyz=-0.1 0 0.2 rpy=0 0.05 0
