Commit message: Made simulation faster by making URDF simpler physically, but not visually

File: robotont_description/xacro/_d435.urdf.xacro (robot description, xacro)
@@ -6,108 +6,98 @@
 aluminum peripherial evaluation case.
 -->
-<robot name="sensor_d435" xmlns:xacro="http://ros.org/wiki/xacro">
-  <xacro:macro name="sensor_d435" params="parent *origin">
-    <xacro:property name="M_PI" value="3.1415926535897931" />
-    <!-- The following values are approximate, and the camera node
+<robot name="sensor_d435"
+    xmlns:xacro="http://ros.org/wiki/xacro">
+    <xacro:macro name="sensor_d435" params="parent *origin">
+        <xacro:property name="M_PI" value="3.1415926535897931" />
+        <!-- The following values are approximate, and the camera node
      publishing TF values with actual calibrated camera extrinsic values -->
-    <xacro:property name="d435_cam_depth_to_left_ir_offset" value="0.0"/>
-    <xacro:property name="d435_cam_depth_to_right_ir_offset" value="-0.050"/>
-    <xacro:property name="d435_cam_depth_to_color_offset" value="0.015"/>
-    <!-- The following values model the aluminum peripherial case for the
+        <xacro:property name="d435_cam_depth_to_left_ir_offset" value="0.0"/>
+        <xacro:property name="d435_cam_depth_to_right_ir_offset" value="-0.050"/>
+        <xacro:property name="d435_cam_depth_to_color_offset" value="0.015"/>
+        <!-- The following values model the aluminum peripherial case for the
   	D435 camera, with the camera joint represented by the actual
   	peripherial camera tripod mount -->
-    <xacro:property name="d435_cam_width" value="0.090"/>
-    <xacro:property name="d435_cam_height" value="0.025"/>
-    <xacro:property name="d435_cam_depth" value="0.02505"/>
-    <xacro:property name="d435_cam_mount_from_center_offset" value="0.0149"/>
-    <!-- The following offset is relative the the physical D435 camera peripherial
+        <xacro:property name="d435_cam_width" value="0.090"/>
+        <xacro:property name="d435_cam_height" value="0.025"/>
+        <xacro:property name="d435_cam_depth" value="0.02505"/>
+        <xacro:property name="d435_cam_mount_from_center_offset" value="0.0149"/>
+        <!-- The following offset is relative the the physical D435 camera peripherial
   	camera tripod mount -->
-    <xacro:property name="d435_cam_depth_px" value="${d435_cam_mount_from_center_offset}"/>
-    <xacro:property name="d435_cam_depth_py" value="0.0175"/>
-    <xacro:property name="d435_cam_depth_pz" value="${d435_cam_height/2}"/>
-    <material name="aluminum">
-	  <color rgba="0.5 0.5 0.5 1"/>
-    </material>
-    <!-- camera body, with origin at bottom screw mount -->
-    <joint name="camera_joint" type="fixed">
-      <xacro:insert_block name="origin" />
-      <parent link="${parent}"/>
-      <child link="camera_link" />
-    </joint>
-    <link name="camera_link">
-      <visual>
-      <origin xyz="${d435_cam_mount_from_center_offset} 0.0 ${d435_cam_height/2}" rpy="${M_PI/2} 0 ${M_PI/2}"/>
-        <geometry>
-          <!-- <box size="${d435_cam_width} ${d435_cam_height} ${d435_cam_depth}"/> -->
-	  <mesh filename="package://realsense2_camera/meshes/d435.dae" />
-          <!--<mesh filename="package://realsense2_camera/meshes/d435/d435.dae" />-->
-        </geometry>
-        <material name="aluminum"/>
-      </visual>
-      <collision>
-        <origin xyz="0.0 0.0 ${d435_cam_height/2}" rpy="0 0 0"/>
-        <geometry>
-        <box size="${d435_cam_depth} ${d435_cam_width} ${d435_cam_height}"/>
-        </geometry>
-      </collision>
-      <inertial>
-        <!-- The following are not reliable values, and should not be used for modeling -->
-        <mass value="0" />
-        <origin xyz="0 0 0" />
-        <inertia ixx="0.003881243" ixy="0.0" ixz="0.0" iyy="0.000498940" iyz="0.0" izz="0.003879257" />
-      </inertial>
-    </link>
-    <!-- camera depth joints and links -->
-    <joint name="camera_depth_joint" type="fixed">
-      <origin xyz="${d435_cam_depth_px} ${d435_cam_depth_py} ${d435_cam_depth_pz}" rpy="0 0 0"/>
-      <parent link="camera_link"/>
-      <child link="camera_depth_frame" />
-    </joint>
-    <link name="camera_depth_frame"/>
-    <joint name="camera_depth_optical_joint" type="fixed">
-      <origin xyz="0 0 0" rpy="${-M_PI/2} 0 ${-M_PI/2}" />
-      <parent link="camera_depth_frame" />
-      <child link="camera_depth_optical_frame" />
-    </joint>
-    <link name="camera_depth_optical_frame"/>
-    <!-- camera left IR joints and links -->
-    <joint name="camera_left_ir_joint" type="fixed">
-      <origin xyz="0 ${d435_cam_depth_to_left_ir_offset} 0" rpy="0 0 0" />
-      <parent link="camera_depth_frame" />
-      <child link="camera_left_ir_frame" />
-    </joint>
-    <link name="camera_left_ir_frame"/>
-    <joint name="camera_left_ir_optical_joint" type="fixed">
-      <origin xyz="0 0 0" rpy="${-M_PI/2} 0 ${-M_PI/2}" />
-      <parent link="camera_left_ir_frame" />
-      <child link="camera_left_ir_optical_frame" />
-    </joint>
-    <link name="camera_left_ir_optical_frame"/>
-    <!-- camera right IR joints and links -->
-    <joint name="camera_right_ir_joint" type="fixed">
-      <origin xyz="0 ${d435_cam_depth_to_right_ir_offset} 0" rpy="0 0 0" />
-      <parent link="camera_depth_frame" />
-      <child link="camera_right_ir_frame" />
-    </joint>
-    <link name="camera_right_ir_frame"/>
-    <joint name="camera_right_ir_optical_joint" type="fixed">
-      <origin xyz="0 0 0" rpy="${-M_PI/2} 0 ${-M_PI/2}" />
-      <parent link="camera_right_ir_frame" />
-      <child link="camera_right_ir_optical_frame" />
-    </joint>
-    <link name="camera_right_ir_optical_frame"/>
-    <!-- camera color joints and links -->
-    <joint name="camera_color_joint" type="fixed">
-      <origin xyz="0 ${d435_cam_depth_to_color_offset} 0" rpy="0 0 0" />
-      <parent link="camera_depth_frame" />
-      <child link="camera_color_frame" />
-    </joint>
-    <link name="camera_color_frame"/>
-    <joint name="camera_color_optical_joint" type="fixed">
-      <origin xyz="0 0 0" rpy="${-M_PI/2} 0 ${-M_PI/2}" />
-      <parent link="camera_color_frame" />
-      <child link="camera_color_optical_frame" />
-    </joint>
-    <link name="camera_color_optical_frame"/>
-  </xacro:macro>
+        <xacro:property name="d435_cam_depth_px" value="${d435_cam_mount_from_center_offset}"/>
+        <xacro:property name="d435_cam_depth_py" value="0.0175"/>
+        <xacro:property name="d435_cam_depth_pz" value="${d435_cam_height/2}"/>
+        <material name="aluminum">
+            <color rgba="0.5 0.5 0.5 1"/>
+        </material>
+        <!-- camera body, with origin at bottom screw mount -->
+        <joint name="camera_joint" type="fixed">
+            <xacro:insert_block name="origin" />
+            <parent link="${parent}"/>
+            <child link="camera_link" />
+        </joint>
+        <link name="camera_link">
+            <visual>
+                <origin xyz="${d435_cam_mount_from_center_offset} 0.0 ${d435_cam_height/2}" rpy="${M_PI/2} 0 ${M_PI/2}"/>
+                <geometry>
+                    <!-- <box size="${d435_cam_width} ${d435_cam_height} ${d435_cam_depth}"/> -->
+                    <mesh filename="package://realsense2_camera/meshes/d435.dae" />
+                    <!--<mesh filename="package://realsense2_camera/meshes/d435/d435.dae" />-->
+                </geometry>
+                <material name="aluminum"/>
+            </visual>
+            <!-- <collision><origin xyz="0.0 0.0 ${d435_cam_height/2}" rpy="0 0 0"/><geometry><box size="${d435_cam_depth} ${d435_cam_width} ${d435_cam_height}"/></geometry></collision> -->
+        </link>
+        <!-- camera depth joints and links -->
+        <joint name="camera_depth_joint" type="fixed">
+            <origin xyz="${d435_cam_depth_px} ${d435_cam_depth_py} ${d435_cam_depth_pz}" rpy="0 0 0"/>
+            <parent link="camera_link"/>
+            <child link="camera_depth_frame" />
+        </joint>
+        <link name="camera_depth_frame"/>
+        <joint name="camera_depth_optical_joint" type="fixed">
+            <origin xyz="0 0 0" rpy="${-M_PI/2} 0 ${-M_PI/2}" />
+            <parent link="camera_depth_frame" />
+            <child link="camera_depth_optical_frame" />
+        </joint>
+        <link name="camera_depth_optical_frame"/>
+        <!-- camera left IR joints and links -->
+        <joint name="camera_left_ir_joint" type="fixed">
+            <origin xyz="0 ${d435_cam_depth_to_left_ir_offset} 0" rpy="0 0 0" />
+            <parent link="camera_depth_frame" />
+            <child link="camera_left_ir_frame" />
+        </joint>
+        <link name="camera_left_ir_frame"/>
+        <joint name="camera_left_ir_optical_joint" type="fixed">
+            <origin xyz="0 0 0" rpy="${-M_PI/2} 0 ${-M_PI/2}" />
+            <parent link="camera_left_ir_frame" />
+            <child link="camera_left_ir_optical_frame" />
+        </joint>
+        <link name="camera_left_ir_optical_frame"/>
+        <!-- camera right IR joints and links -->
+        <joint name="camera_right_ir_joint" type="fixed">
+            <origin xyz="0 ${d435_cam_depth_to_right_ir_offset} 0" rpy="0 0 0" />
+            <parent link="camera_depth_frame" />
+            <child link="camera_right_ir_frame" />
+        </joint>
+        <link name="camera_right_ir_frame"/>
+        <joint name="camera_right_ir_optical_joint" type="fixed">
+            <origin xyz="0 0 0" rpy="${-M_PI/2} 0 ${-M_PI/2}" />
+            <parent link="camera_right_ir_frame" />
+            <child link="camera_right_ir_optical_frame" />
+        </joint>
+        <link name="camera_right_ir_optical_frame"/>
+        <!-- camera color joints and links -->
+        <joint name="camera_color_joint" type="fixed">
+            <origin xyz="0 ${d435_cam_depth_to_color_offset} 0" rpy="0 0 0" />
+            <parent link="camera_depth_frame" />
+            <child link="camera_color_frame" />
+        </joint>
+        <link name="camera_color_frame"/>
+        <joint name="camera_color_optical_joint" type="fixed">
+            <origin xyz="0 0 0" rpy="${-M_PI/2} 0 ${-M_PI/2}" />
+            <parent link="camera_color_frame" />
+            <child link="camera_color_optical_frame" />
+        </joint>
+        <link name="camera_color_optical_frame"/>
+    </xacro:macro>
 </robot>

File: robotont_description/xacro/main.urdf.xacro (robot description, xacro)
@@ -11,5 +11,5 @@
     <link name="base_link">
         <inertial>
-            <mass value="0.07862944645"/>
+            <mass value="3"/>
             <inertia
 			ixx="0.00002035985530754"
@@ -31,6 +31,7 @@
         <collision>
             <geometry>
-                <mesh scale=" 0.001 0.001 0.001" filename="package://robotont_description/meshes/body.stl"/>
+                <mesh scale=" 0.001 0.001 0.001" filename="package://robotont_description/meshes/simplebody.stl"/>
             </geometry>
+            <origin rpy="${pi/2} 0 ${-pi/2}"  xyz="0 0 0"/>
         </collision>
     </link>
@@ -43,5 +44,5 @@
         <origin
 			xyz="0 0 0.013"
-			rpy="0 0 0"
+			rpy="0 0 ${pi/2}"
 		/>
     </joint>
@@ -87,10 +88,4 @@
             </material>
         </visual>
-        <collision>
-            <geometry>
-                <box size="0.11 0.04 0.11"/>
-            </geometry>
-            <origin rpy="0 0 0" xyz="0 0 0"/>
-        </collision>
     </link>
     <joint
@@ -135,5 +130,5 @@
             <odometryFrame>odom</odometryFrame>
             <odometryRate>30.0</odometryRate>
-            <robotBaseFrame>base_footprint</robotBaseFrame>
+            <robotBaseFrame>base_link</robotBaseFrame>
         </plugin>
     </gazebo>
@@ -154,5 +149,5 @@
             <update_rate>10.0</update_rate>
             <camera>
-                <horizontal_fov>${60.0*pi/180.0}</horizontal_fov>
+                <horizontal_fov>${90.0*pi/180.0}</horizontal_fov>
                 <image>
                     <format>B8G8R8</format>

File: robotont_description/xacro/rim.urdf.xacro (robot description, xacro)
@@ -13,5 +13,5 @@
         <link name="rim_${name}_link">
             <inertial>
-                <origin xyz="0 0 -0.000343"/>
+                <origin xyz="0 0 0"/>
                 <mass value="0.00835758"/>
                 <inertia
@@ -34,5 +34,5 @@
             <collision>
                 <geometry>
-                    <mesh filename="package://robotont_description/meshes/rim.stl"/>
+                    <cylinder radius="0.035" length="0.03"/>
                 </geometry>
             </collision>
@@ -164,15 +164,8 @@
 			no_of_roller="6"
 		/>
-        <transmission name="rim_${name}_transmission">
-            <type>transmission_interface/SimpleTransmission</type>
-            <joint name="rim_${name}_joint">
-                <hardwareInterface>hardware_interface/EffortJointInterface</hardwareInterface>
-            </joint>
-            <actuator name="rim_${name}_motor">
-                <mechanicalReduction>1</mechanicalReduction>
-            </actuator>
-        </transmission>
+        <!-- <transmission name="rim_${name}_transmission"><type>transmission_interface/SimpleTransmission</type><joint name="rim_${name}_joint"><hardwareInterface>hardware_interface/EffortJointInterface</hardwareInterface></joint><actuator name="rim_${name}_motor"><mechanicalReduction>1</mechanicalReduction></actuator></transmission> -->
         <gazebo reference="rim_${name}_link">
             <material>Gazebo/DarkGrey</material>
+            <!-- <kp>1000000</kp><kd>100</kd> -->
         </gazebo>
     </xacro:macro>

File: robotont_description/xacro/roller.urdf.xacro (robot description, xacro)
@@ -31,17 +31,12 @@
                 </material>
             </visual>
-            <collision>
-                <geometry>
-                    <mesh scale="0.001 0.001 0.001" filename="package://robotont_description/meshes/roller.stl"/>
-                </geometry>
-            </collision>
         </link>
         <joint
 			name="roller_${name}_rim_${parent}_joint"
-			type="continuous"
+			type="fixed"
 		>
             <parent link="rim_${parent}_link"/>
             <child link="roller_${name}_rim_${parent}_link"/>
-            <axis xyz="1 0 0"/>
+            <!-- <axis xyz="1 0 0"/> -->
             <origin
 				xyz="${radial_dist*sin(-1*z_distance_reflect*(init_angle+offset+no_of_roller*2*pi/7))} ${-radial_dist*cos(-1*z_distance_reflect*(init_angle+offset+no_of_roller*2*pi/7))} ${z_distance*z_distance_reflect}"

Commit message: changed gazebo robot spawn location, fixed realsense stl path in xacro, it is now in realsense2_description

File: robotont_description/xacro/_d435.urdf.xacro (robot description, xacro)
@@ -41,5 +41,5 @@
                 <geometry>
                     <!-- <box size="${d435_cam_width} ${d435_cam_height} ${d435_cam_depth}"/> -->
-                    <mesh filename="package://realsense2_camera/meshes/d435.dae" />
+                    <mesh filename="package://realsense2_description/meshes/d435.dae" />
                     <!--<mesh filename="package://realsense2_camera/meshes/d435/d435.dae" />-->
                 </geometry>
