Commit message: Updated the xacro files to support prefixes

File: robotont_description/xacro/_d435.urdf.xacro (robot description, xacro)
@@ -8,5 +8,5 @@
 <robot name="sensor_d435"
     xmlns:xacro="http://ros.org/wiki/xacro">
-    <xacro:macro name="sensor_d435" params="parent *origin">
+    <xacro:macro name="sensor_d435" params="parent *origin prefix">
         <xacro:property name="M_PI" value="3.1415926535897931" />
         <!-- The following values are approximate, and the camera node
@@ -31,10 +31,10 @@
         </material>
         <!-- camera body, with origin at bottom screw mount -->
-        <joint name="camera_joint" type="fixed">
+        <joint name="${prefix}camera_joint" type="fixed">
             <xacro:insert_block name="origin" />
             <parent link="${parent}"/>
-            <child link="camera_link" />
+            <child link="${prefix}camera_link" />
         </joint>
-        <link name="camera_link">
+        <link name="${prefix}camera_link">
             <visual>
                 <origin xyz="${d435_cam_mount_from_center_offset} 0.0 ${d435_cam_height/2}" rpy="${M_PI/2} 0 ${M_PI/2}"/>
@@ -49,55 +49,55 @@
         </link>
         <!-- camera depth joints and links -->
-        <joint name="camera_depth_joint" type="fixed">
+        <joint name="${prefix}camera_depth_joint" type="fixed">
             <origin xyz="${d435_cam_depth_px} ${d435_cam_depth_py} ${d435_cam_depth_pz}" rpy="0 0 0"/>
-            <parent link="camera_link"/>
-            <child link="camera_depth_frame" />
+            <parent link="${prefix}camera_link"/>
+            <child link="${prefix}camera_depth_frame" />
         </joint>
-        <link name="camera_depth_frame"/>
-        <joint name="camera_depth_optical_joint" type="fixed">
+        <link name="${prefix}camera_depth_frame"/>
+        <joint name="${prefix}camera_depth_optical_joint" type="fixed">
             <origin xyz="0 0 0" rpy="${-M_PI/2} 0 ${-M_PI/2}" />
-            <parent link="camera_depth_frame" />
-            <child link="camera_depth_optical_frame" />
+            <parent link="${prefix}camera_depth_frame" />
+            <child link="${prefix}camera_depth_optical_frame" />
         </joint>
-        <link name="camera_depth_optical_frame"/>
+        <link name="${prefix}camera_depth_optical_frame"/>
         <!-- camera left IR joints and links -->
-        <joint name="camera_left_ir_joint" type="fixed">
+        <joint name="${prefix}camera_left_ir_joint" type="fixed">
             <origin xyz="0 ${d435_cam_depth_to_left_ir_offset} 0" rpy="0 0 0" />
-            <parent link="camera_depth_frame" />
-            <child link="camera_left_ir_frame" />
+            <parent link="${prefix}camera_depth_frame" />
+            <child link="${prefix}camera_left_ir_frame" />
         </joint>
-        <link name="camera_left_ir_frame"/>
-        <joint name="camera_left_ir_optical_joint" type="fixed">
+        <link name="${prefix}camera_left_ir_frame"/>
+        <joint name="${prefix}camera_left_ir_optical_joint" type="fixed">
             <origin xyz="0 0 0" rpy="${-M_PI/2} 0 ${-M_PI/2}" />
-            <parent link="camera_left_ir_frame" />
-            <child link="camera_left_ir_optical_frame" />
+            <parent link="${prefix}camera_left_ir_frame" />
+            <child link="${prefix}camera_left_ir_optical_frame" />
         </joint>
-        <link name="camera_left_ir_optical_frame"/>
+        <link name="${prefix}camera_left_ir_optical_frame"/>
         <!-- camera right IR joints and links -->
-        <joint name="camera_right_ir_joint" type="fixed">
+        <joint name="${prefix}camera_right_ir_joint" type="fixed">
             <origin xyz="0 ${d435_cam_depth_to_right_ir_offset} 0" rpy="0 0 0" />
-            <parent link="camera_depth_frame" />
-            <child link="camera_right_ir_frame" />
+            <parent link="${prefix}camera_depth_frame" />
+            <child link="${prefix}camera_right_ir_frame" />
         </joint>
-        <link name="camera_right_ir_frame"/>
-        <joint name="camera_right_ir_optical_joint" type="fixed">
+        <link name="${prefix}camera_right_ir_frame"/>
+        <joint name="${prefix}camera_right_ir_optical_joint" type="fixed">
             <origin xyz="0 0 0" rpy="${-M_PI/2} 0 ${-M_PI/2}" />
-            <parent link="camera_right_ir_frame" />
-            <child link="camera_right_ir_optical_frame" />
+            <parent link="${prefix}camera_right_ir_frame" />
+            <child link="${prefix}camera_right_ir_optical_frame" />
         </joint>
-        <link name="camera_right_ir_optical_frame"/>
+        <link name="${prefix}camera_right_ir_optical_frame"/>
         <!-- camera color joints and links -->
-        <joint name="camera_color_joint" type="fixed">
+        <joint name="${prefix}camera_color_joint" type="fixed">
             <origin xyz="0 ${d435_cam_depth_to_color_offset} 0" rpy="0 0 0" />
-            <parent link="camera_depth_frame" />
-            <child link="camera_color_frame" />
+            <parent link="${prefix}camera_depth_frame" />
+            <child link="${prefix}camera_color_frame" />
         </joint>
-        <link name="camera_color_frame"/>
-        <joint name="camera_color_optical_joint" type="fixed">
+        <link name="${prefix}camera_color_frame"/>
+        <joint name="${prefix}camera_color_optical_joint" type="fixed">
             <origin xyz="0 0 0" rpy="${-M_PI/2} 0 ${-M_PI/2}" />
-            <parent link="camera_color_frame" />
-            <child link="camera_color_optical_frame" />
+            <parent link="${prefix}camera_color_frame" />
+            <child link="${prefix}camera_color_optical_frame" />
         </joint>
-        <link name="camera_color_optical_frame"/>
+        <link name="${prefix}camera_color_optical_frame"/>
     </xacro:macro>
 </robot>

File: robotont_description/xacro/main.urdf.xacro (robot description, xacro)
@@ -2,10 +2,11 @@
 <robot xmlns:xacro="http://ros.org/wiki/xacro" name="robotont">
     <xacro:arg name="prefix" default=""/>
+    <xacro:property name= "prefix" value="$(arg prefix)"/>
     <xacro:include filename="$(find robotont_description)/xacro/rim.urdf.xacro"/>
     <xacro:include filename="$(find robotont_description)/xacro/_d435.urdf.xacro"/>
     <xacro:property name="wheel_distance" value="0.146" />
     <xacro:property name="wheel_center_height" value="0.021" />
-    <link name="$(arg prefix)base_footprint"/>
-    <link name="$(arg prefix)base_link">
+    <link name="${prefix}base_footprint"/>
+    <link name="${prefix}base_link">
         <inertial>
             <mass value="3"/>
@@ -36,9 +37,9 @@
     </link>
     <joint
-		name="$(arg prefix)base_joint"
+		name="${prefix}base_joint"
 		type="fixed"
 	>
-        <parent link="$(arg prefix)base_footprint" />
-        <child link="$(arg prefix)base_link" />
+        <parent link="${prefix}base_footprint" />
+        <child link="${prefix}base_link" />
         <origin
 			xyz="0 0 0.013"
@@ -66,5 +67,5 @@
 			rpy="0 0 0"
 		/></joint> -->
-    <sensor_d435 parent="$(arg prefix)base_link">
+    <sensor_d435 parent="${prefix}base_link" prefix="${prefix}">
         <origin xyz="-0.12 0 0.21" rpy="0 0 0"/>
     </sensor_d435>
@@ -77,5 +78,5 @@
 		/></joint> -->
     <!-- Computer -->
-    <link name="$(arg prefix)computer_link">
+    <link name="${prefix}computer_link">
         <visual>
             <geometry>
@@ -89,9 +90,9 @@
     </link>
     <joint
-		name="$(arg prefix)computer_joint"
+		name="${prefix}computer_joint"
 		type="fixed"
 	>
-        <parent link="$(arg prefix)base_link" />
-        <child link="$(arg prefix)computer_link" />
+        <parent link="${prefix}base_link" />
+        <child link="${prefix}computer_link" />
         <origin
 			xyz="-0.01 0 0.085"
@@ -106,5 +107,5 @@
 		wheel_distance = "${wheel_distance}"
 		wheel_center_height = "${wheel_center_height}"
-        prefix="$(arg prefix)"
+        prefix="${prefix}"
 	/>
     <xacro:rim_macro
@@ -114,5 +115,5 @@
 		wheel_distance = "${wheel_distance}"
 		wheel_center_height = "${wheel_center_height}"
-        prefix="$(arg prefix)"
+        prefix="${prefix}"
 	/>
     <xacro:rim_macro
@@ -122,5 +123,5 @@
 		wheel_distance = "${wheel_distance}"
 		wheel_center_height = "${wheel_center_height}"
-        prefix="$(arg prefix)"
+        prefix="${prefix}"
 	/>
     <!-- Initialize controller manager and odometry-->
@@ -132,19 +133,19 @@
             <odometryFrame>odom</odometryFrame>
             <odometryRate>30.0</odometryRate>
-            <robotBaseFrame>$(arg prefix)base_footprint</robotBaseFrame>
+            <robotBaseFrame>${prefix}base_footprint</robotBaseFrame>
         </plugin>
     </gazebo>
     <!-- Give materials to links -->
-    <gazebo reference="$(arg prefix)base_link">
+    <gazebo reference="${prefix}base_link">
         <material>Robotont/BlueishTransparent</material>
     </gazebo>
-    <gazebo reference="$(arg prefix)camera_link">
+    <gazebo reference="${prefix}camera_link">
         <material>Gazebo/Grey</material>
     </gazebo>
-    <gazebo reference="$(arg prefix)computer_link">
+    <gazebo reference="${prefix}computer_link">
         <material>Gazebo/Black</material>
     </gazebo>
     <!-- Depth camera plugin -->
-    <gazebo reference="$(arg prefix)camera_link">
+    <gazebo reference="${prefix}camera_link">
         <sensor type="depth" name="camera">
             <always_on>true</always_on>

File: robotont_description/xacro/rim.urdf.xacro (robot description, xacro)
@@ -7,9 +7,6 @@
     <xacro:property name="roller_z_distance" value="0.008" />
     <xacro:property name="roller_init_angle" value="0" />
-    <xacro:macro
-		name="rim_macro"
-		params="name color angle wheel_distance wheel_center_height prefix"
-	>
-        <link name="rim_${name}_link">
+    <xacro:macro name="rim_macro" params="name color angle wheel_distance wheel_center_height prefix">
+		<link name="${prefix}rim_${name}_link">
             <inertial>
                 <origin xyz="0 0 0"/>
@@ -39,9 +36,9 @@
         </link>
         <joint
-			name="rim_${name}_joint"
+			name="${prefix}rim_${name}_joint"
 			type="continuous"
 		>
-            <parent link="$(arg prefix)base_link" />
-            <child link="rim_${name}_link" />
+            <parent link="${prefix}base_link" />
+            <child link="${prefix}rim_${name}_link" />
             <axis xyz="0 0 1"/>
             <origin
@@ -58,4 +55,5 @@
 			init_angle="${roller_init_angle}"
 			no_of_roller="0"
+			prefix="${prefix}"
 		/>
         <xacro:roller_macro
@@ -66,4 +64,5 @@
 			init_angle="${roller_init_angle}"
 			no_of_roller="1"
+			prefix="${prefix}"
 		/>
         <xacro:roller_macro
@@ -74,4 +73,5 @@
 			init_angle="${roller_init_angle}"
 			no_of_roller="2"
+			prefix="${prefix}"
 		/>
         <xacro:roller_macro
@@ -82,4 +82,5 @@
 			init_angle="${roller_init_angle}"
 			no_of_roller="3"
+			prefix="${prefix}"
 		/>
         <xacro:roller_macro
@@ -90,4 +91,5 @@
 			init_angle="${roller_init_angle}"
 			no_of_roller="4"
+			prefix="${prefix}"
 		/>
         <xacro:roller_macro
@@ -98,4 +100,5 @@
 			init_angle="${roller_init_angle}"
 			no_of_roller="5"
+			prefix="${prefix}"
 		/>
         <xacro:roller_macro
@@ -106,4 +109,5 @@
 			init_angle="${roller_init_angle}"
 			no_of_roller="6"
+			prefix="${prefix}"
 		/>
         <!-- Back rollers -->
@@ -115,4 +119,5 @@
 			init_angle="${roller_init_angle}"
 			no_of_roller="0"
+			prefix="${prefix}"
 		/>
         <xacro:roller_macro
@@ -123,4 +128,5 @@
 			init_angle="${roller_init_angle}"
 			no_of_roller="1"
+			prefix="${prefix}"
 		/>
         <xacro:roller_macro
@@ -131,4 +137,5 @@
 			init_angle="${roller_init_angle}"
 			no_of_roller="2"
+			prefix="${prefix}"
 		/>
         <xacro:roller_macro
@@ -139,4 +146,5 @@
 			init_angle="${roller_init_angle}"
 			no_of_roller="3"
+			prefix="${prefix}"
 		/>
         <xacro:roller_macro
@@ -147,4 +155,5 @@
 			init_angle="${roller_init_angle}"
 			no_of_roller="4"
+			prefix="${prefix}"
 		/>
         <xacro:roller_macro
@@ -155,4 +164,5 @@
 			init_angle="${roller_init_angle}"
 			no_of_roller="5"
+			prefix="${prefix}"
 		/>
         <xacro:roller_macro
@@ -163,7 +173,8 @@
 			init_angle="${roller_init_angle}"
 			no_of_roller="6"
+			prefix="${prefix}"
 		/>
         <!-- <transmission name="rim_${name}_transmission"><type>transmission_interface/SimpleTransmission</type><joint name="rim_${name}_joint"><hardwareInterface>hardware_interface/EffortJointInterface</hardwareInterface></joint><actuator name="rim_${name}_motor"><mechanicalReduction>1</mechanicalReduction></actuator></transmission> -->
-        <gazebo reference="rim_${name}_link">
+        <gazebo reference="${prefix}rim_${name}_link">
             <material>Gazebo/DarkGrey</material>
             <!-- <kp>1000000</kp><kd>100</kd> -->

File: robotont_description/xacro/roller.urdf.xacro (robot description, xacro)
@@ -4,5 +4,5 @@
     <xacro:macro
 		name="roller_macro"
-		params="parent radial_dist z_distance z_distance_reflect init_angle no_of_roller"
+		params="parent radial_dist z_distance z_distance_reflect init_angle no_of_roller prefix"
 	>
         <xacro:if value="${z_distance_reflect==-1}">
@@ -14,5 +14,5 @@
             <xacro:property name="offset" value="${pi}" />
         </xacro:unless>
-        <link name="roller_${name}_rim_${parent}_link">
+        <link name="${prefix}roller_${name}_rim_${parent}_link">
             <!-- <inertial><mass value="0.00113845"/><inertia
 					ixx="2.53776e-08"
@@ -33,9 +33,9 @@
         </link>
         <joint
-			name="roller_${name}_rim_${parent}_joint"
+			name="${prefix}roller_${name}_rim_${parent}_joint"
 			type="fixed"
 		>
-            <parent link="rim_${parent}_link"/>
-            <child link="roller_${name}_rim_${parent}_link"/>
+            <parent link="${prefix}rim_${parent}_link"/>
+            <child link="${prefix}roller_${name}_rim_${parent}_link"/>
             <!-- <axis xyz="1 0 0"/> -->
             <origin
@@ -44,5 +44,5 @@
 			/>
         </joint>
-        <gazebo reference="roller_${name}_rim_${parent}_link">
+        <gazebo reference="${prefix}roller_${name}_rim_${parent}_link">
             <material>Robotont/DarkGreen</material>
         </gazebo>
