Commit message: Added realsense camera, which can be used in gazebo. This threw off the center of mass, so driving is broken right now

File: robotont_description/xacro/main.urdf.xacro (robot description, xacro)
@@ -1,8 +1,9 @@
 <?xml version="1.0"?>
 <robot
-    xmlns:xacro="http://www.ros.org/wiki/xacro"
+    xmlns:xacro="http://ros.org/wiki/xacro"
 	name="robotont"
 >
     <xacro:include filename="$(find robotont_description)/xacro/rim.urdf.xacro"/>
+    <xacro:include filename="$(find realsense2_camera)/urdf/_d435.urdf.xacro"/>
     <xacro:property name="wheel_distance" value="0.12" />
     <xacro:property name="wheel_center_height" value="0.021" />
@@ -102,32 +103,36 @@
 		/>
     </joint>
-    <link name="camera_link">
-        <visual>
-            <geometry>
-                <box size="0.1 0.02 0.02"/>
-            </geometry>
-            <origin rpy="0 0 0" xyz="0 0 0"/>
-            <material name="camera_material">
-                <color rgba="0.1 0.1 0.1 1"/>
-            </material>
-        </visual>
-        <collision>
-            <geometry>
-                <box size="0.1 0.02 0.02"/>
-            </geometry>
-            <origin rpy="0 0 0" xyz="0 0 0"/>
-        </collision>
-    </link>
-    <joint
-		name="camera_joint"
+    <link name="camera_base">
+        <visual>
+            <geometry>
+                <box size="0.1 0.02 0.005"/>
+            </geometry>
+            <origin rpy="0 0 0" xyz="0 0 0"/>
+            <material name="boom_material">
+                <color rgba="1 1 1 0.7"/>
+            </material>
+        </visual>
+    </link>
+    <joint
+		name="camera_boom_to_base_joint"
 		type="fixed"
 	>
         <parent link="right_camera_boom" />
-        <child link="camera_link" />
-        <origin
-			xyz="0.05 0.07 0.015"
-			rpy="0 0 0"
-		/>
-    </joint>
+        <child link="camera_base" />
+        <origin
+			xyz="0.0475 0.07 0"
+			rpy="0 0 0"
+		/>
+    </joint>
+    <sensor_d435 parent="camera_base">
+        <origin xyz="0 -0.01 0.011" rpy="${-pi/2} ${-pi/2} 0"/>
+    </sensor_d435>
+    <!-- <link name="camera_link"><origin rpy="0 0 0" xyz="0 0 0"/></link><joint
+		name="camera_base_to_link_joint"
+		type="fixed"
+	><parent link="camera_base" /><child link="camera_link" /><origin
+			xyz="0 0 0.011"
+			rpy="0 0 0"
+		/></joint> -->
     <!-- Computer -->
     <link name="computer_link">
@@ -181,4 +186,5 @@
 		wheel_center_height = "${wheel_center_height}"
 	/>
+    <!-- Initialize controller manager -->
     <gazebo>
         <plugin name="gazebo_ros_control" filename="libgazebo_ros_control.so">
@@ -186,4 +192,5 @@
         </plugin>
     </gazebo>
+    <!-- Give materials to links -->
     <gazebo reference="base_link">
         <material>Robotont/BlueishTransparent</material>
@@ -201,3 +208,44 @@
         <material>Robotont/BlueishTransparent</material>
     </gazebo>
+    <gazebo reference="camera_base">
+        <material>Robotont/BlueishTransparent</material>
+    </gazebo>
+    <!-- Depth camera plugin -->
+    <gazebo reference="camera_link">
+        <sensor type="depth" name="camera">
+            <always_on>true</always_on>
+            <update_rate>30.0</update_rate>
+            <camera>
+                <horizontal_fov>${60.0*pi/180.0}</horizontal_fov>
+                <image>
+                    <format>B8G8R8</format>
+                    <width>640</width>
+                    <height>480</height>
+                </image>
+                <clip>
+                    <near>0.02</near>
+                    <far>8.0</far>
+                </clip>
+            </camera>
+            <plugin name="kinect_camera_controller" filename="libgazebo_ros_openni_kinect.so">
+                <robotNamespace>/</robotNamespace>
+                <cameraName>camera</cameraName>
+                <alwaysOn>true</alwaysOn>
+                <updateRate>0.0</updateRate>
+                <imageTopicName>color/image_raw</imageTopicName>
+                <depthImageTopicName>depth/image_raw</depthImageTopicName>
+                <pointCloudTopicName>depth/points</pointCloudTopicName>
+                <cameraInfoTopicName>color/camera_info</cameraInfoTopicName>
+                <depthImageCameraInfoTopicName>depth/camera_info</depthImageCameraInfoTopicName>
+                <frameName>camera_depth_optical_frame</frameName>
+                <baseline>0.1</baseline>
+                <distortion_k1>0.0</distortion_k1>
+                <distortion_k2>0.0</distortion_k2>
+                <distortion_k3>0.0</distortion_k3>
+                <distortion_t1>0.0</distortion_t1>
+                <distortion_t2>0.0</distortion_t2>
+                <pointCloudCutoff>0.4</pointCloudCutoff>
+            </plugin>
+        </sensor>
+    </gazebo>
 </robot>

File: robotont_description/xacro/rim.urdf.xacro (robot description, xacro)
@@ -1,5 +1,5 @@
 <?xml version="1.0" ?>
 <robot
-    xmlns:xacro="http://www.ros.org/wiki/xacro">
+    xmlns:xacro="http://ros.org/wiki/xacro">
     <xacro:include filename="$(find robotont_description)/xacro/roller.urdf.xacro"/>
     <!-- Roller positioning -->

File: robotont_description/xacro/roller.urdf.xacro (robot description, xacro)
@@ -1,5 +1,5 @@
 <?xml version="1.0" ?>
 <robot
-    xmlns:xacro="http://www.ros.org/wiki/xacro">
+    xmlns:xacro="http://ros.org/wiki/xacro">
     <xacro:macro
 		name="roller_macro"

Commit message: Added correct body.stl, corrigated xacro, driving is broken because of some inertia thing

File: robotont_description/xacro/main.urdf.xacro (robot description, xacro)
@@ -6,10 +6,10 @@
     <xacro:include filename="$(find robotont_description)/xacro/rim.urdf.xacro"/>
     <xacro:include filename="$(find realsense2_camera)/urdf/_d435.urdf.xacro"/>
-    <xacro:property name="wheel_distance" value="0.12" />
+    <xacro:property name="wheel_distance" value="0.146" />
     <xacro:property name="wheel_center_height" value="0.021" />
     <link name="base_footprint"/>
     <link name="base_link">
         <inertial>
-            <mass value="0.07862944645"/>
+            <mass value="0.1"/>
             <inertia
 			ixx="0.00002035985530754"
@@ -31,5 +31,5 @@
         <collision>
             <geometry>
-                <mesh scale="0.001 0.001 0.001" filename="package://robotont_description/meshes/body.stl"/>
+                <mesh scale=" 0.001 0.001 0.001" filename="package://robotont_description/meshes/body.stl"/>
             </geometry>
         </collision>
@@ -43,9 +43,9 @@
         <origin
 			xyz="0 0 0.013"
-			rpy="${pi/2} 0 ${-pi/2}"
+			rpy="0 0 0"
 		/>
     </joint>
     <!-- Camera -->
-    <link name="right_camera_boom">
+    <!-- <link name="right_camera_boom">
         <visual>
             <geometry>
@@ -124,7 +124,7 @@
 			rpy="0 0 0"
 		/>
-    </joint>
-    <sensor_d435 parent="camera_base">
-        <origin xyz="0 -0.01 0.011" rpy="${-pi/2} ${-pi/2} 0"/>
+    </joint> -->
+    <sensor_d435 parent="base_link">
+        <origin xyz="0 0.12 0.21" rpy="0 0 ${-pi/2}"/>
     </sensor_d435>
     <!-- <link name="camera_link"><origin rpy="0 0 0" xyz="0 0 0"/></link><joint
@@ -139,5 +139,5 @@
         <visual>
             <geometry>
-                <box size="0.11 0.04 0.11"/>
+                <box size="0.11 0.11 0.04"/>
             </geometry>
             <origin rpy="0 0 0" xyz="0 0 0"/>
@@ -160,5 +160,5 @@
         <child link="computer_link" />
         <origin
-			xyz="0 0.085 0.01"
+			xyz="0 0.01 0.085"
 			rpy="0 0 0"
 		/>
@@ -201,13 +201,4 @@
     <gazebo reference="computer_link">
         <material>Gazebo/Black</material>
-    </gazebo>
-    <gazebo reference="right_camera_boom">
-        <material>Robotont/BlueishTransparent</material>
-    </gazebo>
-    <gazebo reference="left_camera_boom">
-        <material>Robotont/BlueishTransparent</material>
-    </gazebo>
-    <gazebo reference="camera_base">
-        <material>Robotont/BlueishTransparent</material>
     </gazebo>
     <!-- Depth camera plugin -->

File: robotont_description/xacro/rim.urdf.xacro (robot description, xacro)
@@ -14,5 +14,5 @@
             <inertial>
                 <origin xyz="0 0 -0.000343"/>
-                <mass value="0.00835758"/>
+                <mass value="0.001"/>
                 <inertia
 					ixx="6.63684e-07"
@@ -46,6 +46,6 @@
             <axis xyz="0 0 1"/>
             <origin
-				xyz="${wheel_distance*sin(angle)} ${wheel_center_height} ${wheel_distance*cos(angle)}"
-				rpy="0 ${angle+pi} 0"
+				xyz="${wheel_distance*sin(angle)} ${-wheel_distance*cos(angle)} ${wheel_center_height}"
+				rpy="${pi/2} 0 ${angle+pi}"
 			/>
         </joint>

Commit message: Added simulated odom

File: robotont_description/xacro/main.urdf.xacro (robot description, xacro)
@@ -47,82 +47,23 @@
     </joint>
     <!-- Camera -->
-    <!-- <link name="right_camera_boom">
-        <visual>
-            <geometry>
-                <box size="0.005 0.16 0.01"/>
-            </geometry>
-            <origin rpy="0 0 0" xyz="0 0 0"/>
-            <material name="boom_material">
-                <color rgba="1 1 1 0.7"/>
-            </material>
-        </visual>
-        <collision>
-            <geometry>
-                <box size="0.005 0.16 0.01"/>
-            </geometry>
-            <origin rpy="0 0 0" xyz="0 0 0"/>
-        </collision>
-    </link>
-    <joint
+    <!-- <link name="right_camera_boom"><visual><geometry><box size="0.005 0.16 0.01"/></geometry><origin rpy="0 0 0" xyz="0 0 0"/><material name="boom_material"><color rgba="1 1 1 0.7"/></material></visual><collision><geometry><box size="0.005 0.16 0.01"/></geometry><origin rpy="0 0 0" xyz="0 0 0"/></collision></link><joint
 		name="right_camera_boom_joint"
 		type="fixed"
-	>
-        <parent link="base_link" />
-        <child link="right_camera_boom" />
-        <origin
+	><parent link="base_link" /><child link="right_camera_boom" /><origin
 			xyz="-0.05 0.145 -0.1"
 			rpy="0 0 0"
-		/>
-    </joint>
-    <link name="left_camera_boom">
-        <visual>
-            <geometry>
-                <box size="0.005 0.16 0.01"/>
-            </geometry>
-            <origin rpy="0 0 0" xyz="0 0 0"/>
-            <material name="boom_material">
-                <color rgba="1 1 1 0.7"/>
-            </material>
-        </visual>
-        <collision>
-            <geometry>
-                <box size="0.005 0.16 0.01"/>
-            </geometry>
-            <origin rpy="0 0 0" xyz="0 0 0"/>
-        </collision>
-    </link>
-    <joint
+		/></joint><link name="left_camera_boom"><visual><geometry><box size="0.005 0.16 0.01"/></geometry><origin rpy="0 0 0" xyz="0 0 0"/><material name="boom_material"><color rgba="1 1 1 0.7"/></material></visual><collision><geometry><box size="0.005 0.16 0.01"/></geometry><origin rpy="0 0 0" xyz="0 0 0"/></collision></link><joint
 		name="left_camera_boom_joint"
 		type="fixed"
-	>
-        <parent link="base_link" />
-        <child link="left_camera_boom" />
-        <origin
+	><parent link="base_link" /><child link="left_camera_boom" /><origin
 			xyz="0.05 0.145 -0.1"
 			rpy="0 0 0"
-		/>
-    </joint>
-    <link name="camera_base">
-        <visual>
-            <geometry>
-                <box size="0.1 0.02 0.005"/>
-            </geometry>
-            <origin rpy="0 0 0" xyz="0 0 0"/>
-            <material name="boom_material">
-                <color rgba="1 1 1 0.7"/>
-            </material>
-        </visual>
-    </link>
-    <joint
+		/></joint><link name="camera_base"><visual><geometry><box size="0.1 0.02 0.005"/></geometry><origin rpy="0 0 0" xyz="0 0 0"/><material name="boom_material"><color rgba="1 1 1 0.7"/></material></visual></link><joint
 		name="camera_boom_to_base_joint"
 		type="fixed"
-	>
-        <parent link="right_camera_boom" />
-        <child link="camera_base" />
-        <origin
+	><parent link="right_camera_boom" /><child link="camera_base" /><origin
 			xyz="0.0475 0.07 0"
 			rpy="0 0 0"
-		/>
-    </joint> -->
+		/></joint> -->
     <sensor_d435 parent="base_link">
         <origin xyz="0 0.12 0.21" rpy="0 0 ${-pi/2}"/>
@@ -186,8 +127,18 @@
 		wheel_center_height = "${wheel_center_height}"
 	/>
-    <!-- Initialize controller manager -->
+    <!-- Initialize controller manager and odometry-->
     <gazebo>
         <plugin name="gazebo_ros_control" filename="libgazebo_ros_control.so">
             <robotNamespace>/robotont</robotNamespace>
+        </plugin>
+        <plugin name="p3d_base_controller" filename="libgazebo_ros_p3d.so">
+            <alwaysOn>true</alwaysOn>
+            <updateRate>50.0</updateRate>
+            <bodyName>base_link</bodyName>
+            <topicName>/robotont/odom</topicName>
+            <gaussianNoise>0</gaussianNoise>
+            <frameName>world</frameName>
+            <xyzOffsets>0 0 0</xyzOffsets>
+            <rpyOffsets>0 0 0</rpyOffsets>
         </plugin>
     </gazebo>

Commit message: Working on getting the movement workign again, commit to save progress

File: robotont_description/xacro/main.urdf.xacro (robot description, xacro)
@@ -5,5 +5,5 @@
 >
     <xacro:include filename="$(find robotont_description)/xacro/rim.urdf.xacro"/>
-    <xacro:include filename="$(find realsense2_camera)/urdf/_d435.urdf.xacro"/>
+    <xacro:include filename="$(find robotont_description)/xacro/_d435.urdf.xacro"/>
     <xacro:property name="wheel_distance" value="0.146" />
     <xacro:property name="wheel_center_height" value="0.021" />
@@ -11,5 +11,5 @@
     <link name="base_link">
         <inertial>
-            <mass value="0.1"/>
+            <mass value="0.07862944645"/>
             <inertia
 			ixx="0.00002035985530754"

File: robotont_description/xacro/rim.urdf.xacro (robot description, xacro)
@@ -14,5 +14,5 @@
             <inertial>
                 <origin xyz="0 0 -0.000343"/>
-                <mass value="0.001"/>
+                <mass value="0.00835758"/>
                 <inertia
 					ixx="6.63684e-07"
@@ -173,7 +173,7 @@
             </actuator>
         </transmission>
-		<gazebo reference="rim_${name}_link">
-        	<material>Gazebo/DarkGrey</material>
-    	</gazebo>
+        <gazebo reference="rim_${name}_link">
+            <material>Gazebo/DarkGrey</material>
+        </gazebo>
     </xacro:macro>
 </robot>

Commit message: minor fixes to simulation, discovered that realtime factor is very small

File: robotont_description/xacro/main.urdf.xacro (robot description, xacro)
@@ -134,6 +134,6 @@
         <plugin name="p3d_base_controller" filename="libgazebo_ros_p3d.so">
             <alwaysOn>true</alwaysOn>
-            <updateRate>50.0</updateRate>
-            <bodyName>base_link</bodyName>
+            <updateRate>100.0</updateRate>
+            <bodyName>base_footprint</bodyName>
             <topicName>/robotont/odom</topicName>
             <gaussianNoise>0</gaussianNoise>

File: robotont_description/xacro/roller.urdf.xacro (robot description, xacro)
@@ -15,5 +15,5 @@
         </xacro:unless>
         <link name="roller_${name}_rim_${parent}_link">
-            <inertial>
+            <!-- <inertial>
                 <mass value="0.00113845"/>
                 <inertia
@@ -25,5 +25,5 @@
 					izz="1.47666e-08"
 				/>
-            </inertial>
+            </inertial> -->
             <visual>
                 <geometry>
@@ -55,4 +55,12 @@
             <material>Robotont/DarkGreen</material>
         </gazebo>
+        <gazebo>
+            <plugin name="joint_state_publisher" filename="libgazebo_ros_joint_state_publisher.so">
+                <robotNamespace>/robotont</robotNamespace>
+                <jointName>roller_${name}_rim_${parent}_joint</jointName>
+                <updateRate>20.0</updateRate>
+                <alwaysOn>true</alwaysOn>
+            </plugin>
+        </gazebo>
     </xacro:macro>
 </robot>

Commit message: Changed controller to planar move, maybe is faster

File: robotont_description/xacro/main.urdf.xacro (robot description, xacro)
@@ -128,17 +128,12 @@
 	/>
     <!-- Initialize controller manager and odometry-->
+    <!-- libgazebo_ros_planar_move.so -->
     <gazebo>
-        <plugin name="gazebo_ros_control" filename="libgazebo_ros_control.so">
-            <robotNamespace>/robotont</robotNamespace>
-        </plugin>
-        <plugin name="p3d_base_controller" filename="libgazebo_ros_p3d.so">
-            <alwaysOn>true</alwaysOn>
-            <updateRate>100.0</updateRate>
-            <bodyName>base_footprint</bodyName>
-            <topicName>/robotont/odom</topicName>
-            <gaussianNoise>0</gaussianNoise>
-            <frameName>world</frameName>
-            <xyzOffsets>0 0 0</xyzOffsets>
-            <rpyOffsets>0 0 0</rpyOffsets>
+        <plugin name="robotont_controller" filename="libgazebo_ros_planar_move.so">
+            <commandTopic>/robotont/cmd_vel</commandTopic>
+            <odometryTopic>/robotont/odom</odometryTopic>
+            <odometryFrame>odom</odometryFrame>
+            <odometryRate>30.0</odometryRate>
+            <robotBaseFrame>base_footprint</robotBaseFrame>
         </plugin>
     </gazebo>
@@ -157,5 +152,5 @@
         <sensor type="depth" name="camera">
             <always_on>true</always_on>
-            <update_rate>30.0</update_rate>
+            <update_rate>10.0</update_rate>
             <camera>
                 <horizontal_fov>${60.0*pi/180.0}</horizontal_fov>

File: robotont_description/xacro/roller.urdf.xacro (robot description, xacro)
@@ -15,7 +15,5 @@
         </xacro:unless>
         <link name="roller_${name}_rim_${parent}_link">
-            <!-- <inertial>
-                <mass value="0.00113845"/>
-                <inertia
+            <!-- <inertial><mass value="0.00113845"/><inertia
 					ixx="2.53776e-08"
 					ixy="0"
@@ -24,6 +22,5 @@
 					iyz="0"
 					izz="1.47666e-08"
-				/>
-            </inertial> -->
+				/></inertial> -->
             <visual>
                 <geometry>
@@ -55,12 +52,4 @@
             <material>Robotont/DarkGreen</material>
         </gazebo>
-        <gazebo>
-            <plugin name="joint_state_publisher" filename="libgazebo_ros_joint_state_publisher.so">
-                <robotNamespace>/robotont</robotNamespace>
-                <jointName>roller_${name}_rim_${parent}_joint</jointName>
-                <updateRate>20.0</updateRate>
-                <alwaysOn>true</alwaysOn>
-            </plugin>
-        </gazebo>
     </xacro:macro>
 </robot>

Commit message: minor fixes in transforms

File: robotont_description/xacro/main.urdf.xacro (robot description, xacro)
@@ -28,4 +28,5 @@
                 <color rgba="1 1 1 0.8"/>
             </material>
+            <origin rpy="0 0 ${pi/2}"  xyz="0 0 0"/>
         </visual>
         <collision>
@@ -33,5 +34,5 @@
                 <mesh scale=" 0.001 0.001 0.001" filename="package://robotont_description/meshes/simplebody.stl"/>
             </geometry>
-            <origin rpy="${pi/2} 0 ${-pi/2}"  xyz="0 0 0"/>
+            <origin rpy="${pi/2} 0 0"  xyz="0 0 0"/>
         </collision>
     </link>
@@ -44,5 +45,5 @@
         <origin
 			xyz="0 0 0.013"
-			rpy="0 0 ${pi/2}"
+			rpy="0 0 0"
 		/>
     </joint>
@@ -68,5 +69,5 @@
 		/></joint> -->
     <sensor_d435 parent="base_link">
-        <origin xyz="0 0.12 0.21" rpy="0 0 ${-pi/2}"/>
+        <origin xyz="-0.12 0 0.21" rpy="0 0 0"/>
     </sensor_d435>
     <!-- <link name="camera_link"><origin rpy="0 0 0" xyz="0 0 0"/></link><joint
@@ -96,5 +97,5 @@
         <child link="computer_link" />
         <origin
-			xyz="0 0.01 0.085"
+			xyz="-0.01 0 0.085"
 			rpy="0 0 0"
 		/>
@@ -104,5 +105,5 @@
 		name="back"
 		color="0 0.3 0"
-		angle="${pi}"
+		angle="${3*pi/2}"
 		wheel_distance = "${wheel_distance}"
 		wheel_center_height = "${wheel_center_height}"
@@ -111,5 +112,5 @@
 		name="right"
 		color="0 0.3 0"
-		angle="${-1/3*pi}"
+		angle="${-1/3*pi + pi/2}"
 		wheel_distance = "${wheel_distance}"
 		wheel_center_height = "${wheel_center_height}"
@@ -118,5 +119,5 @@
 		name="left"
 		color="0 0.3 0"
-		angle="${1/3*pi}"
+		angle="${1/3*pi + pi/2}"
 		wheel_distance = "${wheel_distance}"
 		wheel_center_height = "${wheel_center_height}"
@@ -130,5 +131,5 @@
             <odometryFrame>odom</odometryFrame>
             <odometryRate>30.0</odometryRate>
-            <robotBaseFrame>base_link</robotBaseFrame>
+            <robotBaseFrame>base_footprint</robotBaseFrame>
         </plugin>
     </gazebo>
