Commit message: Add prefix to the main and rim xacro files

File: robotont_description/xacro/main.urdf.xacro (robot description, xacro)
@@ -1,13 +1,11 @@
 <?xml version="1.0"?>
-<robot
-    xmlns:xacro="http://ros.org/wiki/xacro"
-	name="robotont"
->
+<robot xmlns:xacro="http://ros.org/wiki/xacro" name="robotont">
+    <xacro:arg name="prefix" default=""/>
     <xacro:include filename="$(find robotont_description)/xacro/rim.urdf.xacro"/>
     <xacro:include filename="$(find robotont_description)/xacro/_d435.urdf.xacro"/>
     <xacro:property name="wheel_distance" value="0.146" />
     <xacro:property name="wheel_center_height" value="0.021" />
-    <link name="base_footprint"/>
-    <link name="base_link">
+    <link name="$(arg prefix)base_footprint"/>
+    <link name="$(arg prefix)base_link">
         <inertial>
             <mass value="3"/>
@@ -38,9 +36,9 @@
     </link>
     <joint
-		name="base_joint"
+		name="$(arg prefix)base_joint"
 		type="fixed"
 	>
-        <parent link="base_footprint" />
-        <child link="base_link" />
+        <parent link="$(arg prefix)base_footprint" />
+        <child link="$(arg prefix)base_link" />
         <origin
 			xyz="0 0 0.013"
@@ -68,5 +66,5 @@
 			rpy="0 0 0"
 		/></joint> -->
-    <sensor_d435 parent="base_link">
+    <sensor_d435 parent="$(arg prefix)base_link">
         <origin xyz="-0.12 0 0.21" rpy="0 0 0"/>
     </sensor_d435>
@@ -79,5 +77,5 @@
 		/></joint> -->
     <!-- Computer -->
-    <link name="computer_link">
+    <link name="$(arg prefix)computer_link">
         <visual>
             <geometry>
@@ -91,9 +89,9 @@
     </link>
     <joint
-		name="computer_joint"
+		name="$(arg prefix)computer_joint"
 		type="fixed"
 	>
-        <parent link="base_link" />
-        <child link="computer_link" />
+        <parent link="$(arg prefix)base_link" />
+        <child link="$(arg prefix)computer_link" />
         <origin
 			xyz="-0.01 0 0.085"
@@ -108,4 +106,5 @@
 		wheel_distance = "${wheel_distance}"
 		wheel_center_height = "${wheel_center_height}"
+        prefix="$(arg prefix)"
 	/>
     <xacro:rim_macro
@@ -115,4 +114,5 @@
 		wheel_distance = "${wheel_distance}"
 		wheel_center_height = "${wheel_center_height}"
+        prefix="$(arg prefix)"
 	/>
     <xacro:rim_macro
@@ -122,4 +122,5 @@
 		wheel_distance = "${wheel_distance}"
 		wheel_center_height = "${wheel_center_height}"
+        prefix="$(arg prefix)"
 	/>
     <!-- Initialize controller manager and odometry-->
@@ -131,19 +132,19 @@
             <odometryFrame>odom</odometryFrame>
             <odometryRate>30.0</odometryRate>
-            <robotBaseFrame>base_footprint</robotBaseFrame>
+            <robotBaseFrame>$(arg prefix)base_footprint</robotBaseFrame>
         </plugin>
     </gazebo>
     <!-- Give materials to links -->
-    <gazebo reference="base_link">
+    <gazebo reference="$(arg prefix)base_link">
         <material>Robotont/BlueishTransparent</material>
     </gazebo>
-    <gazebo reference="camera_link">
+    <gazebo reference="$(arg prefix)camera_link">
         <material>Gazebo/Grey</material>
     </gazebo>
-    <gazebo reference="computer_link">
+    <gazebo reference="$(arg prefix)computer_link">
         <material>Gazebo/Black</material>
     </gazebo>
     <!-- Depth camera plugin -->
-    <gazebo reference="camera_link">
+    <gazebo reference="$(arg prefix)camera_link">
         <sensor type="depth" name="camera">
             <always_on>true</always_on>

File: robotont_description/xacro/rim.urdf.xacro (robot description, xacro)
@@ -9,5 +9,5 @@
     <xacro:macro
 		name="rim_macro"
-		params="name color angle wheel_distance wheel_center_height"
+		params="name color angle wheel_distance wheel_center_height prefix"
 	>
         <link name="rim_${name}_link">
@@ -42,5 +42,5 @@
 			type="continuous"
 		>
-            <parent link="base_link" />
+            <parent link="$(arg prefix)base_link" />
             <child link="rim_${name}_link" />
             <axis xyz="0 0 1"/>

Commit message: Revert some changes in main and rim xacro files

File: robotont_description/xacro/main.urdf.xacro (robot description, xacro)
@@ -1,11 +1,10 @@
 <?xml version="1.0"?>
 <robot xmlns:xacro="http://ros.org/wiki/xacro" name="robotont">
-    <xacro:arg name="prefix" default=""/>
     <xacro:include filename="$(find robotont_description)/xacro/rim.urdf.xacro"/>
     <xacro:include filename="$(find robotont_description)/xacro/_d435.urdf.xacro"/>
     <xacro:property name="wheel_distance" value="0.146" />
     <xacro:property name="wheel_center_height" value="0.021" />
-    <link name="$(arg prefix)base_footprint"/>
-    <link name="$(arg prefix)base_link">
+    <link name="base_footprint"/>
+    <link name="base_link">
         <inertial>
             <mass value="3"/>
@@ -36,9 +35,9 @@
     </link>
     <joint
-		name="$(arg prefix)base_joint"
+		name="base_joint"
 		type="fixed"
 	>
-        <parent link="$(arg prefix)base_footprint" />
-        <child link="$(arg prefix)base_link" />
+        <parent link="base_footprint" />
+        <child link="base_link" />
         <origin
 			xyz="0 0 0.013"
@@ -66,5 +65,5 @@
 			rpy="0 0 0"
 		/></joint> -->
-    <sensor_d435 parent="$(arg prefix)base_link">
+    <sensor_d435 parent="base_link">
         <origin xyz="-0.12 0 0.21" rpy="0 0 0"/>
     </sensor_d435>
@@ -77,5 +76,5 @@
 		/></joint> -->
     <!-- Computer -->
-    <link name="$(arg prefix)computer_link">
+    <link name="computer_link">
         <visual>
             <geometry>
@@ -89,9 +88,9 @@
     </link>
     <joint
-		name="$(arg prefix)computer_joint"
+		name="computer_joint"
 		type="fixed"
 	>
-        <parent link="$(arg prefix)base_link" />
-        <child link="$(arg prefix)computer_link" />
+        <parent link="base_link" />
+        <child link="computer_link" />
         <origin
 			xyz="-0.01 0 0.085"
@@ -106,5 +105,4 @@
 		wheel_distance = "${wheel_distance}"
 		wheel_center_height = "${wheel_center_height}"
-        prefix="$(arg prefix)"
 	/>
     <xacro:rim_macro
@@ -114,5 +112,4 @@
 		wheel_distance = "${wheel_distance}"
 		wheel_center_height = "${wheel_center_height}"
-        prefix="$(arg prefix)"
 	/>
     <xacro:rim_macro
@@ -122,5 +119,4 @@
 		wheel_distance = "${wheel_distance}"
 		wheel_center_height = "${wheel_center_height}"
-        prefix="$(arg prefix)"
 	/>
     <!-- Initialize controller manager and odometry-->
@@ -132,19 +128,19 @@
             <odometryFrame>odom</odometryFrame>
             <odometryRate>30.0</odometryRate>
-            <robotBaseFrame>$(arg prefix)base_footprint</robotBaseFrame>
+            <robotBaseFrame>base_footprint</robotBaseFrame>
         </plugin>
     </gazebo>
     <!-- Give materials to links -->
-    <gazebo reference="$(arg prefix)base_link">
+    <gazebo reference="base_link">
         <material>Robotont/BlueishTransparent</material>
     </gazebo>
-    <gazebo reference="$(arg prefix)camera_link">
+    <gazebo reference="camera_link">
         <material>Gazebo/Grey</material>
     </gazebo>
-    <gazebo reference="$(arg prefix)computer_link">
+    <gazebo reference="computer_link">
         <material>Gazebo/Black</material>
     </gazebo>
     <!-- Depth camera plugin -->
-    <gazebo reference="$(arg prefix)camera_link">
+    <gazebo reference="camera_link">
         <sensor type="depth" name="camera">
             <always_on>true</always_on>

File: robotont_description/xacro/rim.urdf.xacro (robot description, xacro)
@@ -9,5 +9,5 @@
     <xacro:macro
 		name="rim_macro"
-		params="name color angle wheel_distance wheel_center_height prefix"
+		params="name color angle wheel_distance wheel_center_height"
 	>
         <link name="rim_${name}_link">
@@ -42,5 +42,5 @@
 			type="continuous"
 		>
-            <parent link="$(arg prefix)base_link" />
+            <parent link="base_link" />
             <child link="rim_${name}_link" />
             <axis xyz="0 0 1"/>

Commit message: Updated xacro files to support prefixes

File: robotont_description/xacro/main.urdf.xacro (robot description, xacro)
@@ -1,20 +1,12 @@
 <?xml version="1.0"?>
 <robot xmlns:xacro="http://ros.org/wiki/xacro" name="robotont">
-<<<<<<< HEAD
     <xacro:arg name="prefix" default=""/>
     <xacro:property name= "prefix" value="$(arg prefix)"/>
-=======
->>>>>>> 268d3a832c0d9b758c1fe4e2acb1133db5699fd1
     <xacro:include filename="$(find robotont_description)/xacro/rim.urdf.xacro"/>
     <xacro:include filename="$(find robotont_description)/xacro/_d435.urdf.xacro"/>
     <xacro:property name="wheel_distance" value="0.146" />
     <xacro:property name="wheel_center_height" value="0.021" />
-<<<<<<< HEAD
     <link name="${prefix}base_footprint"/>
     <link name="${prefix}base_link">
-=======
-    <link name="base_footprint"/>
-    <link name="base_link">
->>>>>>> 268d3a832c0d9b758c1fe4e2acb1133db5699fd1
         <inertial>
             <mass value="3"/>
@@ -45,5 +37,4 @@
     </link>
     <joint
-<<<<<<< HEAD
 		name="${prefix}base_joint"
 		type="fixed"
@@ -51,11 +42,4 @@
         <parent link="${prefix}base_footprint" />
         <child link="${prefix}base_link" />
-=======
-		name="base_joint"
-		type="fixed"
-	>
-        <parent link="base_footprint" />
-        <child link="base_link" />
->>>>>>> 268d3a832c0d9b758c1fe4e2acb1133db5699fd1
         <origin
 			xyz="0 0 0.013"
@@ -83,9 +67,5 @@
 			rpy="0 0 0"
 		/></joint> -->
-<<<<<<< HEAD
     <sensor_d435 parent="${prefix}base_link" prefix="${prefix}">
-=======
-    <sensor_d435 parent="base_link">
->>>>>>> 268d3a832c0d9b758c1fe4e2acb1133db5699fd1
         <origin xyz="-0.12 0 0.21" rpy="0 0 0"/>
     </sensor_d435>
@@ -98,9 +78,5 @@
 		/></joint> -->
     <!-- Computer -->
-<<<<<<< HEAD
     <link name="${prefix}computer_link">
-=======
-    <link name="computer_link">
->>>>>>> 268d3a832c0d9b758c1fe4e2acb1133db5699fd1
         <visual>
             <geometry>
@@ -114,5 +90,4 @@
     </link>
     <joint
-<<<<<<< HEAD
 		name="${prefix}computer_joint"
 		type="fixed"
@@ -120,11 +95,4 @@
         <parent link="${prefix}base_link" />
         <child link="${prefix}computer_link" />
-=======
-		name="computer_joint"
-		type="fixed"
-	>
-        <parent link="base_link" />
-        <child link="computer_link" />
->>>>>>> 268d3a832c0d9b758c1fe4e2acb1133db5699fd1
         <origin
 			xyz="-0.01 0 0.085"
@@ -139,8 +107,5 @@
 		wheel_distance = "${wheel_distance}"
 		wheel_center_height = "${wheel_center_height}"
-<<<<<<< HEAD
         prefix="${prefix}"
-=======
->>>>>>> 268d3a832c0d9b758c1fe4e2acb1133db5699fd1
 	/>
     <xacro:rim_macro
@@ -150,8 +115,5 @@
 		wheel_distance = "${wheel_distance}"
 		wheel_center_height = "${wheel_center_height}"
-<<<<<<< HEAD
         prefix="${prefix}"
-=======
->>>>>>> 268d3a832c0d9b758c1fe4e2acb1133db5699fd1
 	/>
     <xacro:rim_macro
@@ -161,8 +123,5 @@
 		wheel_distance = "${wheel_distance}"
 		wheel_center_height = "${wheel_center_height}"
-<<<<<<< HEAD
         prefix="${prefix}"
-=======
->>>>>>> 268d3a832c0d9b758c1fe4e2acb1133db5699fd1
 	/>
     <!-- Initialize controller manager and odometry-->
@@ -174,5 +133,4 @@
             <odometryFrame>odom</odometryFrame>
             <odometryRate>30.0</odometryRate>
-<<<<<<< HEAD
             <robotBaseFrame>${prefix}base_footprint</robotBaseFrame>
         </plugin>
@@ -190,21 +148,4 @@
     <!-- Depth camera plugin -->
     <gazebo reference="${prefix}camera_link">
-=======
-            <robotBaseFrame>base_footprint</robotBaseFrame>
-        </plugin>
-    </gazebo>
-    <!-- Give materials to links -->
-    <gazebo reference="base_link">
-        <material>Robotont/BlueishTransparent</material>
-    </gazebo>
-    <gazebo reference="camera_link">
-        <material>Gazebo/Grey</material>
-    </gazebo>
-    <gazebo reference="computer_link">
-        <material>Gazebo/Black</material>
-    </gazebo>
-    <!-- Depth camera plugin -->
-    <gazebo reference="camera_link">
->>>>>>> 268d3a832c0d9b758c1fe4e2acb1133db5699fd1
         <sensor type="depth" name="camera">
             <always_on>true</always_on>

File: robotont_description/xacro/rim.urdf.xacro (robot description, xacro)
@@ -7,14 +7,6 @@
     <xacro:property name="roller_z_distance" value="0.008" />
     <xacro:property name="roller_init_angle" value="0" />
-<<<<<<< HEAD
     <xacro:macro name="rim_macro" params="name color angle wheel_distance wheel_center_height prefix">
 		<link name="${prefix}rim_${name}_link">
-=======
-    <xacro:macro
-		name="rim_macro"
-		params="name color angle wheel_distance wheel_center_height"
-	>
-        <link name="rim_${name}_link">
->>>>>>> 268d3a832c0d9b758c1fe4e2acb1133db5699fd1
             <inertial>
                 <origin xyz="0 0 0"/>
@@ -47,11 +39,6 @@
 			type="continuous"
 		>
-<<<<<<< HEAD
             <parent link="${prefix}base_link" />
             <child link="${prefix}rim_${name}_link" />
-=======
-            <parent link="base_link" />
-            <child link="rim_${name}_link" />
->>>>>>> 268d3a832c0d9b758c1fe4e2acb1133db5699fd1
             <axis xyz="0 0 1"/>
             <origin
